Commit message: m

File: src/envs/bullet_cartpole/double_cartpole_goal/double_hangpole.urdf (robot description, URDF)
Before this commit: robot physics, 4 links, 3 joints
Joints:
- joint slider_to_cart: limit lower=-3 upper=3 effort=1000.0 velocity=5 -> lower=-3 upper=3 effort=100.0 velocity=5
- joint swing_1: limit lower=-2 upper=2 effort=1000.0 velocity=10 -> lower=-30 upper=30 effort=200.0 velocity=10
- joint swing_2: limit lower=-2 upper=2 effort=1000.0 velocity=10 -> lower=-2 upper=2 effort=100.0 velocity=1

Commit message: m

File: src/envs/bullet_cartpole/double_cartpole_goal/double_hangpole.urdf (robot description, URDF)
Before this commit: robot physics, 4 links, 3 joints
Joints:
- joint swing_2: origin xyz=0.0 0.0 -0.5 -> xyz=0.0 0.0 0.5
