Commit message: m

File: src/envs/bullet_cartpole/cartpole/cartpole.urdf (robot description, URDF)
Before this commit: robot physics, 4 links, 3 joints
Links:
- removed link pole_2
- link pole_1: geometry visual box size=0.05 0.05 1.0
Joints:
- removed joint swing_2
- joint swing_1: limit lower=-30 upper=30 effort=200.0 velocity=10 -> lower=-30 upper=30 effort=200.0 velocity=5

File: src/envs/bullet_cartpole/hangpole_goal/target.urdf (robot description, URDF)
Before this commit: robot target, 1 links, 0 joints
Links:
- removed link goal
- added link pole, mass 0.0; visual sphere radius=0.1
