Commit message: m

File: src/envs/bullet_cartpole/double_cartpole_swingup_goal_variable/double_hangpole.urdf (robot description, URDF)
Before this commit: robot physics, 3 links, 2 joints
Links:
- added link pole_2, mass 1; visual box size=0.05 0.05 0.5
- link pole_1: geometry visual box size=0.05 0.05 0.5
Joints:
- added joint swing_2: type continuous, parent pole_1, child pole_2, origin xyz=0.0 0.0 -0.5, axis 0 1 0, limit lower=-2 upper=2 effort=1000.0 velocity=10
- joint slider_to_cart: limit lower=-3 upper=3 effort=100.0 velocity=5 -> lower=-3 upper=3 effort=1000.0 velocity=5
- joint swing_1: limit lower=-30 upper=30 effort=200.0 velocity=5 -> lower=-2 upper=2 effort=1000.0 velocity=10

File: src/envs/bullet_cartpole/tmp/cartpole.urdf (robot description, URDF)
Before this commit: robot physics, 3 links, 2 joints
Links:
- removed link pole_1
- added link sphere, mass 1.0; collision box size=0.05 0.05 1.0; visual sphere radius=0.1
Joints:
- removed joint swing_1
- added joint swing: type continuous, parent cart, child sphere, origin xyz=0.0 0.0 0, axis 0 1 0, limit lower=-2 upper=2 effort=1000.0 velocity=10
- joint slider_to_cart: limit lower=-3 upper=3 effort=100.0 velocity=5 -> lower=-3 upper=3 effort=1000.0 velocity=5

File: src/envs/bullet_cartpole/tmp/hangpole.urdf (robot description, URDF)
Before this commit: robot physics, 3 links, 2 joints
Links:
- removed link pole_1
- added link sphere, mass 1.0; collision box size=0.05 0.05 1.0; visual sphere radius=0.1
Joints:
- removed joint swing_1
- added joint swing: type continuous, parent cart, child sphere, origin xyz=0.0 0.0 0, axis 0 1 0, limit lower=-2 upper=2 effort=1000.0 velocity=10
- joint slider_to_cart: limit lower=-3 upper=3 effort=100.0 velocity=5 -> lower=-3 upper=3 effort=1000.0 velocity=5

File: src/envs/bullet_cartpole/tmp/hangpole_vl.urdf (robot description, URDF)
Before this commit: robot physics, 3 links, 2 joints
Links:
- removed link pole_1
- added link sphere, mass 1.0; collision box size=0.05 0.05 1.0; visual sphere radius=0.1
Joints:
- removed joint swing_1
- added joint swing: type continuous, parent cart, child sphere, origin xyz=0.0 0.0 0, axis 0 1 0, limit lower=-2 upper=2 effort=1000.0 velocity=10
- joint slider_to_cart: limit lower=-3 upper=3 effort=100.0 velocity=5 -> lower=-3 upper=3 effort=1000.0 velocity=5
