Commit message: Both straight and perlin train without contacts. Perlin is ok-ish performance on real platform but rough on body angles.

File: src/envs/bullet_nexabot/hexapod/hexapod_wip.urdf (robot description, URDF)
Before this commit: robot quadruped, 19 links, 18 joints
Links:
- link tibia_fl: geometry collision cylinder length=0.132 radius=0.015; visual cylinder length=0.132 radius=0.015
- link tibia_fr: geometry collision cylinder length=0.132 radius=0.015; visual cylinder length=0.132 radius=0.015
- link tibia_ml: geometry collision cylinder length=0.132 radius=0.015; visual cylinder length=0.132 radius=0.015
- link tibia_mr: geometry collision cylinder length=0.132 radius=0.015; visual cylinder length=0.132 radius=0.015
- link tibia_rl: geometry collision cylinder length=0.132 radius=0.015; visual cylinder length=0.132 radius=0.015
- link tibia_rr: geometry collision cylinder length=0.132 radius=0.015; visual cylinder length=0.132 radius=0.015
- link torso: geometry collision box size=0.20 0.9 0.01; visual box size=0.20 0.12 0.01
Joints:
- joint femur_tibia_fl: origin xyz=0.0 0.066 0 rpy=-0.7854 0 0 -> xyz=0.0 0.066 -0.014 rpy=-0.7854 0 0
- joint femur_tibia_fr: origin xyz=0.0 0.066 0 rpy=-0.7854 0 0 -> xyz=0.0 0.066 -0.014 rpy=-0.7854 0 0
- joint femur_tibia_ml: origin xyz=0.0 0.066 0 rpy=-0.7854 0 0 -> xyz=0.0 0.066 -0.014 rpy=-0.7854 0 0
- joint femur_tibia_mr: origin xyz=0.0 0.066 0 rpy=-0.7854 0 0 -> xyz=0.0 0.066 -0.014 rpy=-0.7854 0 0
- joint femur_tibia_rl: origin xyz=0.0 0.066 0 rpy=-0.7854 0 0 -> xyz=0.0 0.066 -0.014 rpy=-0.7854 0 0
- joint femur_tibia_rr: origin xyz=0.0 0.066 0 rpy=-0.7854 0 0 -> xyz=0.0 0.066 -0.014 rpy=-0.7854 0 0

File: src/envs/bullet_nexabot/hexapod/hexapod_wip_scaled.urdf (robot description, URDF)
Before this commit: robot quadruped, 19 links, 18 joints
Links:
- link tibia_fl: geometry collision cylinder length=0.132 radius=0.015; visual cylinder length=0.132 radius=0.015
- link tibia_fr: geometry collision cylinder length=0.132 radius=0.015; visual cylinder length=0.132 radius=0.015
- link tibia_ml: geometry collision cylinder length=0.132 radius=0.015; visual cylinder length=0.132 radius=0.015
- link tibia_mr: geometry collision cylinder length=0.132 radius=0.015; visual cylinder length=0.132 radius=0.015
- link tibia_rl: geometry collision cylinder length=0.132 radius=0.015; visual cylinder length=0.132 radius=0.015
- link tibia_rr: geometry collision cylinder length=0.132 radius=0.015; visual cylinder length=0.132 radius=0.015
- link torso: geometry collision box size=0.20 0.9 0.01; visual box size=0.20 0.12 0.01
Joints:
- joint coxa_femur_fl: limit lower=-1.6 upper=-0.6 effort=1.4 velocity=1 -> lower=-5.0 upper=5.0 effort=1.4 velocity=1
- joint coxa_femur_fr: limit lower=-1.6 upper=-0.6 effort=1.4 velocity=1 -> lower=-5.0 upper=5.0 effort=1.4 velocity=1
- joint coxa_femur_ml: limit lower=-1.6 upper=-0.6 effort=1.4 velocity=1 -> lower=-5.0 upper=5.0 effort=1.4 velocity=1
- joint coxa_femur_mr: limit lower=-1.6 upper=-0.6 effort=1.4 velocity=1 -> lower=-5.0 upper=5.0 effort=1.4 velocity=1
- joint coxa_femur_rl: limit lower=-1.6 upper=-0.6 effort=1.4 velocity=1 -> lower=-5.0 upper=5.0 effort=1.4 velocity=1
- joint coxa_femur_rr: limit lower=-1.6 upper=-0.6 effort=1.4 velocity=1 -> lower=-5.0 upper=5.0 effort=1.4 velocity=1
- joint femur_tibia_fl: limit lower=0.9 upper=1.9 effort=1.4 velocity=1 -> lower=-5.0 upper=5.0 effort=1.4 velocity=1; origin xyz=0.0 0.066 0 rpy=-0.7854 0 0 -> xyz=0.0 0.066 -0.014 rpy=-0.7854 0 0
- joint femur_tibia_fr: limit lower=0.9 upper=1.9 effort=1.4 velocity=1 -> lower=-5.0 upper=5.0 effort=1.4 velocity=1; origin xyz=0.0 0.066 0 rpy=-0.7854 0 0 -> xyz=0.0 0.066 -0.014 rpy=-0.7854 0 0
- joint femur_tibia_ml: limit lower=0.9 upper=1.9 effort=1.4 velocity=1 -> lower=-5.0 upper=5.0 effort=1.4 velocity=1; origin xyz=0.0 0.066 0 rpy=-0.7854 0 0 -> xyz=0.0 0.066 -0.014 rpy=-0.7854 0 0
- joint femur_tibia_mr: limit lower=0.9 upper=1.9 effort=1.4 velocity=1 -> lower=-5.0 upper=5.0 effort=1.4 velocity=1; origin xyz=0.0 0.066 0 rpy=-0.7854 0 0 -> xyz=0.0 0.066 -0.014 rpy=-0.7854 0 0
- joint femur_tibia_rl: limit lower=0.9 upper=1.9 effort=1.4 velocity=1 -> lower=-5.0 upper=5.0 effort=1.4 velocity=1; origin xyz=0.0 0.066 0 rpy=-0.7854 0 0 -> xyz=0.0 0.066 -0.014 rpy=-0.7854 0 0
- joint femur_tibia_rr: limit lower=0.9 upper=1.9 effort=1.4 velocity=1 -> lower=-5.0 upper=5.0 effort=1.4 velocity=1; origin xyz=0.0 0.066 0 rpy=-0.7854 0 0 -> xyz=0.0 0.066 -0.014 rpy=-0.7854 0 0
- joint torso_coxa_fl: limit lower=-0.4 upper=0.4 effort=1.4 velocity=1 -> lower=-5.0 upper=5.0 effort=1.4 velocity=1
- joint torso_coxa_fr: limit lower=-0.4 upper=0.4 effort=1.4 velocity=1 -> lower=-5.0 upper=5.0 effort=1.4 velocity=1
- joint torso_coxa_ml: limit lower=-0.4 upper=0.4 effort=1.4 velocity=1 -> lower=-5.0 upper=5.0 effort=1.4 velocity=1
- joint torso_coxa_mr: limit lower=-0.4 upper=0.4 effort=1.4 velocity=1 -> lower=-5.0 upper=5.0 effort=1.4 velocity=1
- joint torso_coxa_rl: limit lower=-0.4 upper=0.4 effort=1.4 velocity=1 -> lower=-5.0 upper=5.0 effort=1.4 velocity=1
- joint torso_coxa_rr: limit lower=-0.4 upper=0.4 effort=1.4 velocity=1 -> lower=-5.0 upper=5.0 effort=1.4 velocity=1

Commit message: Add tb log dirs

File: src/envs/bullet_nexabot/hexapod/hexapod_wip.urdf (robot description, URDF)
Before this commit: robot quadruped, 19 links, 18 joints
Links:
- link coxa_fl: geometry collision cylinder length=0.052 radius=0.015; visual cylinder length=0.052 radius=0.015
- link coxa_fr: geometry collision cylinder length=0.052 radius=0.015; visual cylinder length=0.052 radius=0.015
- link coxa_ml: geometry collision cylinder length=0.052 radius=0.015; visual cylinder length=0.052 radius=0.015
- link coxa_mr: geometry collision cylinder length=0.052 radius=0.015; visual cylinder length=0.052 radius=0.015
- link coxa_rl: geometry collision cylinder length=0.052 radius=0.015; visual cylinder length=0.052 radius=0.015
- link coxa_rr: geometry collision cylinder length=0.052 radius=0.015; visual cylinder length=0.052 radius=0.015

File: src/envs/bullet_nexabot/hexapod/hexapod_wip_normal.urdf (robot description, URDF)
Before this commit: robot quadruped, 19 links, 18 joints
Links:
- link coxa_fl: geometry collision cylinder length=0.052 radius=0.015; visual cylinder length=0.052 radius=0.015
- link coxa_fr: geometry collision cylinder length=0.052 radius=0.015; visual cylinder length=0.052 radius=0.015
- link coxa_ml: geometry collision cylinder length=0.052 radius=0.015; visual cylinder length=0.052 radius=0.015
- link coxa_mr: geometry collision cylinder length=0.052 radius=0.015; visual cylinder length=0.052 radius=0.015
- link coxa_rl: geometry collision cylinder length=0.052 radius=0.015; visual cylinder length=0.052 radius=0.015
- link coxa_rr: geometry collision cylinder length=0.052 radius=0.015; visual cylinder length=0.052 radius=0.015
