Commit message: c

File: src/envs/bullet_nexabot/hexapod/hexapod_wip_wide_range.urdf (robot description, URDF)
Before this commit: robot quadruped, 19 links, 18 joints
Links:
- link coxa_fl: geometry collision cylinder length=0.052 radius=0.015; visual cylinder length=0.052 radius=0.015
- link coxa_fr: geometry collision cylinder length=0.052 radius=0.015; visual cylinder length=0.052 radius=0.015
- link coxa_ml: geometry collision cylinder length=0.052 radius=0.015; visual cylinder length=0.052 radius=0.015
- link coxa_mr: geometry collision cylinder length=0.052 radius=0.015; visual cylinder length=0.052 radius=0.015
- link coxa_rl: geometry collision cylinder length=0.052 radius=0.015; visual cylinder length=0.052 radius=0.015
- link coxa_rr: geometry collision cylinder length=0.052 radius=0.015; visual cylinder length=0.052 radius=0.015
