Commit message: m

File: src/envs/bullet_nexabot/hexapod/hexapod.urdf (robot description, URDF)
Before this commit: robot quadruped, 19 links, 18 joints
Links:
- link torso: mass 1.5 -> 1.8; geometry collision box size=0.28 0.14 0.08; visual box size=0.28 0.14 0.08

Commit message: m

File: src/envs/bullet_nexabot/hexapod/hexapod.urdf (robot description, URDF)
Before this commit: robot quadruped, 19 links, 18 joints
Links:
- link coxa_fl: geometry visual cylinder length=0.052 radius=0.015
- link coxa_fr: geometry visual cylinder length=0.052 radius=0.015
- link coxa_ml: geometry visual cylinder length=0.052 radius=0.015
- link coxa_mr: geometry visual cylinder length=0.052 radius=0.015
- link coxa_rl: geometry visual cylinder length=0.052 radius=0.015
- link coxa_rr: geometry visual cylinder length=0.052 radius=0.015
- link femur_fl: geometry visual cylinder length=0.066 radius=0.015
- link femur_fr: geometry visual cylinder length=0.066 radius=0.015
- link femur_ml: geometry visual cylinder length=0.066 radius=0.015
- link femur_mr: geometry visual cylinder length=0.066 radius=0.015
- link femur_rl: geometry visual cylinder length=0.066 radius=0.015
- link femur_rr: geometry visual cylinder length=0.066 radius=0.015
- link tibia_fl: geometry collision cylinder length=0.095 radius=0.015; visual cylinder length=0.095 radius=0.015
- link tibia_fr: geometry collision cylinder length=0.095 radius=0.015; visual cylinder length=0.095 radius=0.015
- link tibia_ml: geometry collision cylinder length=0.095 radius=0.015; visual cylinder length=0.095 radius=0.015
- link tibia_mr: geometry collision cylinder length=0.095 radius=0.015; visual cylinder length=0.095 radius=0.015
- link tibia_rl: geometry collision cylinder length=0.095 radius=0.015; visual cylinder length=0.095 radius=0.015
- link tibia_rr: geometry collision cylinder length=0.095 radius=0.015; visual cylinder length=0.095 radius=0.015
- link torso: geometry collision box size=0.20 0.12 0.01; visual box size=0.20 0.12 0.01
Joints:
- joint coxa_femur_fl: origin xyz=0.0 0.01 0 -> xyz=0.0 0.052 0
- joint coxa_femur_fr: axis 1 0 0 -> -1 0 0; origin xyz=0.0 -0.01 0 -> xyz=0.0 0.052 0
- joint coxa_femur_ml: origin xyz=0.0 0.01 0 -> xyz=0.0 0.052 0
- joint coxa_femur_mr: axis 1 0 0 -> -1 0 0; origin xyz=0.0 -0.01 0 -> xyz=0.0 0.052 0
- joint coxa_femur_rl: origin xyz=0.0 0.01 0 -> xyz=0.0 0.052 0
- joint coxa_femur_rr: axis 1 0 0 -> -1 0 0; origin xyz=0.0 -0.01 0 -> xyz=0.0 0.052 0
- joint femur_tibia_fl: origin xyz=0.0 0.06 0 -> xyz=0.0 0.066 0 rpy=-0.7854 0 0
- joint femur_tibia_fr: axis 1 0 0 -> -1 0 0; origin xyz=0.0 -0.06 0 -> xyz=0.0 0.066 0 rpy=-0.7854 0 0
- joint femur_tibia_ml: origin xyz=0.0 0.06 0 -> xyz=0.0 0.066 0 rpy=-0.7854 0 0
- joint femur_tibia_mr: axis 1 0 0 -> -1 0 0; origin xyz=0.0 -0.06 0 -> xyz=0.0 0.066 0 rpy=-0.7854 0 0
- joint femur_tibia_rl: origin xyz=0.0 0.06 0 -> xyz=0.0 0.066 0 rpy=-0.7854 0 0
- joint femur_tibia_rr: axis 1 0 0 -> -1 0 0; origin xyz=0.0 -0.06 0 -> xyz=0.0 0.066 0 rpy=-0.7854 0 0
- joint torso_coxa_fl: origin xyz=0.05 0.05 0 rpy=0 0 -0.7 -> xyz=0.12 0.06 0 rpy=0 0 -0.7854
- joint torso_coxa_fr: axis 0 0 1 -> 0 0 -1; origin xyz=0.05 -0.05 0 rpy=0 0 0.7 -> xyz=0.12 -0.06 0 rpy=0 0 -2.3562
- joint torso_coxa_ml: origin xyz=0.05 0.05 0 rpy=0 0 -0.7 -> xyz=0.0 0.1 0 rpy=0 0 0
- joint torso_coxa_mr: axis 0 0 1 -> 0 0 -1; origin xyz=0.05 -0.05 0 rpy=0 0 0.7 -> xyz=0 -0.1 0 rpy=0 0 -3.1416
- joint torso_coxa_rl: origin xyz=-0.05 0.05 0 rpy=0 0 0.7 -> xyz=-0.12 0.06 0 rpy=0 0 0.7854
- joint torso_coxa_rr: axis 0 0 1 -> 0 0 -1; origin xyz=-0.05 -0.05 0 rpy=0 0 -0.7 -> xyz=-0.12 -0.06 0 rpy=0 0 2.3561

Commit message: m

File: src/envs/bullet_nexabot/hexapod/hexapod.urdf (robot description, URDF)
Before this commit: robot quadruped, 19 links, 18 joints
Joints:
- joint torso_coxa_fr: axis 0 0 -1 -> 0 0 1
- joint torso_coxa_mr: axis 0 0 -1 -> 0 0 1
- joint torso_coxa_rr: axis 0 0 -1 -> 0 0 1

Commit message: m

File: src/envs/bullet_nexabot/hexapod/hexapod.urdf (robot description, URDF)
Before this commit: robot quadruped, 19 links, 18 joints
Joints:
- joint torso_coxa_fl: axis 0 0 -1 -> 0 0 1
- joint torso_coxa_ml: axis 0 0 -1 -> 0 0 1
- joint torso_coxa_rl: axis 0 0 -1 -> 0 0 1

Commit message: Fix demo funs

File: src/envs/bullet_nexabot/hexapod/hexapod.urdf (robot description, URDF)
Before this commit: robot quadruped, 19 links, 18 joints
Joints:
- joint coxa_femur_fl: limit lower=-3 upper=3 effort=2.0 velocity=5 -> lower=-3 upper=3 effort=1.4 velocity=1
- joint coxa_femur_fr: limit lower=-3 upper=3 effort=2.0 velocity=5 -> lower=-3 upper=3 effort=1.4 velocity=1
- joint coxa_femur_ml: limit lower=-3 upper=3 effort=2.0 velocity=5 -> lower=-3 upper=3 effort=1.4 velocity=1
- joint coxa_femur_mr: limit lower=-3 upper=3 effort=2.0 velocity=5 -> lower=-3 upper=3 effort=1.4 velocity=1
- joint coxa_femur_rl: limit lower=-3 upper=3 effort=2.0 velocity=5 -> lower=-3 upper=3 effort=1.4 velocity=1
- joint coxa_femur_rr: limit lower=-3 upper=3 effort=2.0 velocity=5 -> lower=-3 upper=3 effort=1.4 velocity=1
- joint femur_tibia_fl: limit lower=-3 upper=3 effort=2.0 velocity=5 -> lower=-3 upper=3 effort=1.4 velocity=1
- joint femur_tibia_fr: limit lower=-3 upper=3 effort=2.0 velocity=5 -> lower=-3 upper=3 effort=1.4 velocity=1
- joint femur_tibia_ml: limit lower=-3 upper=3 effort=2.0 velocity=5 -> lower=-3 upper=3 effort=1.4 velocity=1
- joint femur_tibia_mr: limit lower=-3 upper=3 effort=2.0 velocity=5 -> lower=-3 upper=3 effort=1.4 velocity=1
- joint femur_tibia_rl: limit lower=-3 upper=3 effort=2.0 velocity=5 -> lower=-3 upper=3 effort=1.4 velocity=1
- joint femur_tibia_rr: limit lower=-3 upper=3 effort=2.0 velocity=5 -> lower=-3 upper=3 effort=1.4 velocity=1
- joint torso_coxa_fl: limit lower=-3 upper=3 effort=2.0 velocity=5 -> lower=-3 upper=3 effort=1.4 velocity=1
- joint torso_coxa_fr: limit lower=-3 upper=3 effort=2.0 velocity=5 -> lower=-3 upper=3 effort=1.4 velocity=1
- joint torso_coxa_ml: limit lower=-3 upper=3 effort=2.0 velocity=5 -> lower=-3 upper=3 effort=1.4 velocity=1
- joint torso_coxa_mr: limit lower=-3 upper=3 effort=2.0 velocity=5 -> lower=-3 upper=3 effort=1.4 velocity=1
- joint torso_coxa_rl: limit lower=-3 upper=3 effort=2.0 velocity=5 -> lower=-3 upper=3 effort=1.4 velocity=1
- joint torso_coxa_rr: limit lower=-3 upper=3 effort=2.0 velocity=5 -> lower=-3 upper=3 effort=1.4 velocity=1

Commit message: Fix demo funs

File: src/envs/bullet_nexabot/hexapod/hexapod.urdf (robot description, URDF)
Before this commit: robot quadruped, 19 links, 18 joints
Joints:
- joint torso_coxa_fr: axis 0 0 1 -> 0 0 -1
- joint torso_coxa_mr: axis 0 0 1 -> 0 0 -1
- joint torso_coxa_rr: axis 0 0 1 -> 0 0 -1

Commit message: Cleanup

File: src/envs/bullet_nexabot/hexapod/hexapod.urdf (robot description, URDF)
Before this commit: robot quadruped, 19 links, 18 joints
Links:
- link coxa_fl: geometry collision cylinder length=0.052 radius=0.015; visual cylinder length=0.052 radius=0.015
- link coxa_fr: geometry collision cylinder length=0.052 radius=0.015; visual cylinder length=0.052 radius=0.015
- link coxa_ml: geometry collision cylinder length=0.052 radius=0.015; visual cylinder length=0.052 radius=0.015
- link coxa_mr: geometry collision cylinder length=0.052 radius=0.015; visual cylinder length=0.052 radius=0.015
- link coxa_rl: geometry collision cylinder length=0.052 radius=0.015; visual cylinder length=0.052 radius=0.015
- link coxa_rr: geometry collision cylinder length=0.052 radius=0.015; visual cylinder length=0.052 radius=0.015
- link tibia_fl: geometry collision cylinder length=0.132 radius=0.015; visual cylinder length=0.132 radius=0.015
- link tibia_fr: geometry collision cylinder length=0.132 radius=0.015; visual cylinder length=0.132 radius=0.015
- link tibia_ml: geometry collision cylinder length=0.132 radius=0.015; visual cylinder length=0.132 radius=0.015
- link tibia_mr: geometry collision cylinder length=0.132 radius=0.015; visual cylinder length=0.132 radius=0.015
- link tibia_rl: geometry collision cylinder length=0.132 radius=0.015; visual cylinder length=0.132 radius=0.015
- link tibia_rr: geometry collision cylinder length=0.132 radius=0.015; visual cylinder length=0.132 radius=0.015
- link torso: geometry collision box size=0.20 0.9 0.01; visual box size=0.20 0.12 0.01
Joints:
- joint femur_tibia_fl: origin xyz=0.0 0.066 0 rpy=-0.7854 0 0 -> xyz=0.0 0.066 -0.014 rpy=-0.7854 0 0
- joint femur_tibia_fr: origin xyz=0.0 0.066 0 rpy=-0.7854 0 0 -> xyz=0.0 0.066 -0.014 rpy=-0.7854 0 0
- joint femur_tibia_ml: origin xyz=0.0 0.066 0 rpy=-0.7854 0 0 -> xyz=0.0 0.066 -0.014 rpy=-0.7854 0 0
- joint femur_tibia_mr: origin xyz=0.0 0.066 0 rpy=-0.7854 0 0 -> xyz=0.0 0.066 -0.014 rpy=-0.7854 0 0
- joint femur_tibia_rl: origin xyz=0.0 0.066 0 rpy=-0.7854 0 0 -> xyz=0.0 0.066 -0.014 rpy=-0.7854 0 0
- joint femur_tibia_rr: origin xyz=0.0 0.066 0 rpy=-0.7854 0 0 -> xyz=0.0 0.066 -0.014 rpy=-0.7854 0 0
