Commit message: m

File: src/envs/bullet_cartpole/hangpole_goal_cont_variable/hangpole_goal_cont_variable.urdf (robot description, URDF)
Before this commit: robot physics, 4 links, 3 joints
Links:
- link pole: geometry visual box size=0.05 0.05 1.0
- link weight: geometry visual sphere radius=0.1
Joints:
- joint cart_to_pole: limit (none) -> lower=-30 upper=30 effort=200.0 velocity=5

Commit message: Cleanup

File: src/envs/bullet_cartpole/hangpole_goal_cont_variable/hangpole_goal_cont_variable.urdf (robot description, URDF)
Before this commit: robot physics, 4 links, 3 joints
Joints:
- joint slider_to_cart: limit lower=-15 upper=15 effort=1000.0 velocity=5 -> lower=-3 upper=3 effort=1000.0 velocity=5

Commit message: Revised hangpole

File: src/envs/bullet_cartpole/hangpole_goal_cont_variable/hangpole_goal_cont_variable.urdf (robot description, URDF)
Before this commit: robot physics, 4 links, 3 joints
Links:
- link cart: mass 1 -> 0.3
- link pole: mass 1 -> 0.01
Joints:
- joint sphere_to_pole: axis 0 0 1 -> 0 0 -1
