Commit message: quad env with randomization

File: src/envs/bullet_buggy/buggy.urdf (robot description, URDF)
Before this commit: robot quadrotor, 9 links, 8 joints
Links:
- removed link base
- removed link boom_fl
- removed link boom_fr
- removed link boom_rl
- removed link boom_rr
- removed link motor_fl
- removed link motor_fr
- removed link motor_rl
- removed link motor_rr
- added link base_link, mass .1
- added link camera_link, mass 1e-5
- added link chassis, mass .1; visual mesh filename=meshes/chassis.STL
- added link chassis_inertia, mass 4.0
- added link laser, mass 0.130; collision box size=0.1 0.1 0.1; visual mesh filename=meshes/hokuyo.obj
- added link left_front_wheel, mass 0.34055; collision cylinder length=0.045 radius=0.05; visual mesh filename=meshes/left_front_wheel.obj
- added link left_rear_wheel, mass 0.34055; collision cylinder length=0.045 radius=0.05; visual mesh filename=meshes/left_rear_wheel.obj
- added link left_steering_hinge, mass 0.100; visual mesh filename=meshes/left_steering_hinge.STL
- added link right_front_wheel, mass 0.34055; collision cylinder length=0.045 radius=0.05; visual mesh filename=meshes/right_front_wheel.obj
- added link right_rear_wheel, mass 0.34055; collision cylinder length=0.045 radius=0.05; visual mesh filename=meshes/right_rear_wheel.obj
- added link right_steering_hinge, mass 0.100; visual mesh filename=meshes/right_steering_hinge.STL
- added link zed_camera_link, mass 1e-5; collision box size=0.033 0.175 0.030; visual box size=0.033 0.175 0.030
- added link zed_camera_right_link, mass 1e-5
Joints:
- removed joint base_boom_fl
- removed joint base_boom_fr
- removed joint base_boom_rl
- removed joint base_boom_rr
- removed joint boom_motor_fl
- removed joint boom_motor_fr
- removed joint boom_motor_rl
- removed joint boom_motor_rr
- added joint base_link_joint: type fixed, parent base_link, child chassis, origin xyz=0 0 0.05 rpy=0 0 0
- added joint chassis_inertia_joint: type fixed, parent chassis, child chassis_inertia, origin xyz=0 0 0 rpy=0 0 0
- added joint hokuyo_joint: type fixed, parent chassis, child laser, origin xyz=0.265 0.0 0.075 rpy=0 0 0, axis 0 0 1
- added joint left_front_wheel_joint: type continuous, parent left_steering_hinge, child left_front_wheel, origin xyz=0 0 0 rpy=1.5708 0 0, axis 0 0 -1, limit effort=10 velocity=100
- added joint left_rear_wheel_joint: type continuous, parent chassis, child left_rear_wheel, origin xyz=0 0.1 0 rpy=1.5708 0 0, axis 0 0 -1, limit effort=10 velocity=100
- added joint left_steering_hinge_joint: type revolute, parent chassis, child left_steering_hinge, origin xyz=0.325 0.1 0 rpy=0 1.5708 0, axis -1 0 0, limit lower=-1.0 upper=1.0 effort=10 velocity=100
- added joint right_front_wheel_joint: type continuous, parent right_steering_hinge, child right_front_wheel, origin xyz=0 0 0 rpy=1.5708 0 0, axis 0 0 -1, limit effort=10 velocity=100
- added joint right_rear_wheel_joint: type continuous, parent chassis, child right_rear_wheel, origin xyz=0 -0.1 0 rpy=1.5708 0 0, axis 0 0 -1, limit effort=10 velocity=100
- added joint right_steering_hinge_joint: type continuous, parent chassis, child right_steering_hinge, origin xyz=0.325 -0.1 0 rpy=0 1.5708 0, axis -1 0 0, limit lower=-1.0 upper=1.0 effort=10 velocity=100
- added joint zed_camera_joint: type fixed, parent chassis, child zed_camera_link, origin xyz=0.390 0 0.04 rpy=0 0 0, axis 0 0 1
- added joint zed_camera_left_joint: type fixed, parent zed_camera_link, child camera_link, origin xyz=0 0.06 0 rpy=0 0 0, axis 0 0 1
- added joint zed_camera_right_joint: type fixed, parent zed_camera_link, child zed_camera_right_link, origin xyz=0 -0.06 0 rpy=0 0 0, axis 0 0 1
