Commit message: m

File: src/envs/bullet_nexabot/quadruped/quadruped.urdf (robot description, URDF)
Before this commit: robot physics, 3 links, 2 joints
Links:
- removed link cart
- removed link pole_1
- removed link slideBar
- added link femur_lr, mass 0; visual cylinder length=0.1 radius=0.01
- added link torso, mass 0; visual box size=0.2 0.1 0.05
Joints:
- removed joint slider_to_cart
- removed joint swing_1
- added joint torso_femur_lr: type prismatic, parent torso, child femur_lr, origin xyz=0.0 0.0 0.0, axis 1 0 0, limit lower=-3 upper=3 effort=100.0 velocity=5

Commit message: m

File: src/envs/bullet_nexabot/quadruped/quadruped.urdf (robot description, URDF)
Before this commit: robot quadruped, 2 links, 1 joints
Links:
- removed link femur_lr
- added link coxa_fr, mass 1; visual cylinder length=0.02 radius=0.01
- added link femur_fr, mass 1; visual cylinder length=0.1 radius=0.01
- added link tibia_fr, mass 1; visual cylinder length=0.1 radius=0.01
- link torso: mass 0 -> 1; geometry visual box size=0.1 0.1 0.05
Joints:
- removed joint torso_femur_lr
- added joint coxa_femur_fr: type revolute, parent coxa_fr, child femur_fr, origin xyz=0.0 -0.10 0, axis 0 0 1, limit lower=-2 upper=2 effort=100.0 velocity=5
- added joint coxa_tibia_fr: type revolute, parent coxa_fr, child tibia_fr, origin xyz=0.0 -0.10 0, axis 0 0 1, limit lower=-2 upper=2 effort=100.0 velocity=5
- added joint torso_coxa_fr: type revolute, parent torso, child coxa_fr, origin xyz=0.05 -0.05 0, axis 0 0 1, limit lower=-2 upper=2 effort=100.0 velocity=5

Commit message: m

File: src/envs/bullet_nexabot/quadruped/quadruped.urdf (robot description, URDF)
Before this commit: robot quadruped, 4 links, 3 joints
Joints:
- removed joint coxa_tibia_fr
- added joint femur_tibia_fr: type revolute, parent femur_fr, child tibia_fr, origin xyz=0.0 -0.10 0, axis 0 0 1, limit lower=-2 upper=2 effort=100.0 velocity=5
- joint coxa_femur_fr: origin xyz=0.0 -0.10 0 -> xyz=0.0 -0.01 0

Commit message: Fix demo funs

File: src/envs/bullet_nexabot/quadruped/quadruped.urdf (robot description, URDF)
Before this commit: robot quadruped, 4 links, 3 joints
Links:
- added link coxa_fl, mass 1; visual cylinder length=0.02 radius=0.01
- added link coxa_rl, mass 1; visual cylinder length=0.02 radius=0.01
- added link coxa_rr, mass 1; visual cylinder length=0.02 radius=0.01
- added link femur_fl, mass 1; visual cylinder length=0.1 radius=0.01
- added link femur_rl, mass 1; visual cylinder length=0.1 radius=0.01
- added link femur_rr, mass 1; visual cylinder length=0.1 radius=0.01
- added link tibia_fl, mass 1; collision cylinder length=0.1 radius=0.01; visual cylinder length=0.1 radius=0.01
- added link tibia_rl, mass 1; collision cylinder length=0.1 radius=0.01; visual cylinder length=0.1 radius=0.01
- added link tibia_rr, mass 1; collision cylinder length=0.1 radius=0.01; visual cylinder length=0.1 radius=0.01
- link tibia_fr: geometry collision cylinder length=0.1 radius=0.01; visual cylinder length=0.1 radius=0.01
- link torso: geometry collision box size=0.1 0.1 0.05; visual box size=0.1 0.1 0.05
Joints:
- added joint coxa_femur_fl: type revolute, parent coxa_fl, child femur_fl, origin xyz=0.0 0.01 0, axis 1 0 0, limit lower=-2 upper=2 effort=100.0 velocity=5
- added joint coxa_femur_rl: type revolute, parent coxa_rl, child femur_rl, origin xyz=0.0 0.01 0, axis 1 0 0, limit lower=-2 upper=2 effort=100.0 velocity=5
- added joint coxa_femur_rr: type revolute, parent coxa_rr, child femur_rr, origin xyz=0.0 -0.01 0, axis 1 0 0, limit lower=-2 upper=2 effort=100.0 velocity=5
- added joint femur_tibia_fl: type revolute, parent femur_fl, child tibia_fl, origin xyz=0.0 0.10 0, axis 1 0 0, limit lower=-2 upper=2 effort=100.0 velocity=5
- added joint femur_tibia_rl: type revolute, parent femur_rl, child tibia_rl, origin xyz=0.0 0.10 0, axis 1 0 0, limit lower=-2 upper=2 effort=100.0 velocity=5
- added joint femur_tibia_rr: type revolute, parent femur_rr, child tibia_rr, origin xyz=0.0 -0.10 0, axis 1 0 0, limit lower=-2 upper=2 effort=100.0 velocity=5
- added joint torso_coxa_fl: type revolute, parent torso, child coxa_fl, origin xyz=0.05 0.05 0, axis 0 0 1, limit lower=-2 upper=2 effort=100.0 velocity=5
- added joint torso_coxa_rl: type revolute, parent torso, child coxa_rl, origin xyz=-0.05 0.05 0, axis 0 0 1, limit lower=-2 upper=2 effort=100.0 velocity=5
- added joint torso_coxa_rr: type revolute, parent torso, child coxa_rr, origin xyz=-0.05 -0.05 0, axis 0 0 1, limit lower=-2 upper=2 effort=100.0 velocity=5
- joint coxa_femur_fr: axis 0 0 1 -> 1 0 0
- joint femur_tibia_fr: axis 0 0 1 -> 1 0 0

Commit message: Fix demo funs

File: src/envs/bullet_nexabot/quadruped/quadruped.urdf (robot description, URDF)
Before this commit: robot quadruped, 13 links, 12 joints
Links:
- link coxa_fl: mass 1 -> 0.1
- link coxa_fr: mass 1 -> 0.1
- link coxa_rl: mass 1 -> 0.1
- link coxa_rr: mass 1 -> 0.1
- link femur_fl: mass 1 -> 0.1
- link femur_fr: mass 1 -> 0.1
- link femur_rl: mass 1 -> 0.1
- link femur_rr: mass 1 -> 0.1
- link tibia_fl: mass 1 -> 0.1
- link tibia_fr: mass 1 -> 0.1
- link tibia_rl: mass 1 -> 0.1
- link tibia_rr: mass 1 -> 0.1
- link torso: mass 1 -> 1.5
Joints:
- joint coxa_femur_fl: axis 1 0 0 -> -1 0 0
- joint coxa_femur_rl: axis 1 0 0 -> -1 0 0
- joint femur_tibia_fl: axis 1 0 0 -> -1 0 0
- joint femur_tibia_rl: axis 1 0 0 -> -1 0 0
- joint torso_coxa_fl: axis 0 0 1 -> 0 0 -1
- joint torso_coxa_rl: axis 0 0 1 -> 0 0 -1

Commit message: Fix demo funs

File: src/envs/bullet_nexabot/quadruped/quadruped.urdf (robot description, URDF)
Before this commit: robot quadruped, 13 links, 12 joints
Joints:
- joint coxa_femur_fl: limit lower=-2 upper=2 effort=100.0 velocity=5 -> lower=-3 upper=3 effort=100.0 velocity=5
- joint coxa_femur_fr: limit lower=-2 upper=2 effort=100.0 velocity=5 -> lower=-3 upper=3 effort=100.0 velocity=5
- joint coxa_femur_rl: limit lower=-2 upper=2 effort=100.0 velocity=5 -> lower=-3 upper=3 effort=100.0 velocity=5
- joint coxa_femur_rr: limit lower=-2 upper=2 effort=100.0 velocity=5 -> lower=-3 upper=3 effort=100.0 velocity=5
- joint femur_tibia_fl: limit lower=-2 upper=2 effort=100.0 velocity=5 -> lower=-3 upper=3 effort=100.0 velocity=5
- joint femur_tibia_fr: limit lower=-2 upper=2 effort=100.0 velocity=5 -> lower=-3 upper=3 effort=100.0 velocity=5
- joint femur_tibia_rl: limit lower=-2 upper=2 effort=100.0 velocity=5 -> lower=-3 upper=3 effort=100.0 velocity=5
- joint femur_tibia_rr: limit lower=-2 upper=2 effort=100.0 velocity=5 -> lower=-3 upper=3 effort=100.0 velocity=5
- joint torso_coxa_fl: limit lower=-2 upper=2 effort=100.0 velocity=5 -> lower=-3 upper=3 effort=100.0 velocity=5
- joint torso_coxa_fr: limit lower=-2 upper=2 effort=100.0 velocity=5 -> lower=-3 upper=3 effort=100.0 velocity=5
- joint torso_coxa_rl: limit lower=-2 upper=2 effort=100.0 velocity=5 -> lower=-3 upper=3 effort=100.0 velocity=5
- joint torso_coxa_rr: limit lower=-2 upper=2 effort=100.0 velocity=5 -> lower=-3 upper=3 effort=100.0 velocity=5

Commit message: Fix demo funs

File: src/envs/bullet_nexabot/quadruped/quadruped.urdf (robot description, URDF)
Before this commit: robot quadruped, 13 links, 12 joints
Links:
- link femur_fl: geometry visual cylinder length=0.06 radius=0.01
- link femur_fr: geometry visual cylinder length=0.06 radius=0.01
- link femur_rl: geometry visual cylinder length=0.06 radius=0.01
- link femur_rr: geometry visual cylinder length=0.06 radius=0.01
- link tibia_fl: geometry collision cylinder length=0.12 radius=0.01; visual cylinder length=0.12 radius=0.01
- link tibia_fr: geometry collision cylinder length=0.12 radius=0.01; visual cylinder length=0.12 radius=0.01
- link tibia_rl: geometry collision cylinder length=0.12 radius=0.01; visual cylinder length=0.12 radius=0.01
- link tibia_rr: geometry collision cylinder length=0.12 radius=0.01; visual cylinder length=0.12 radius=0.01
Joints:
- joint femur_tibia_fl: origin xyz=0.0 0.10 0 -> xyz=0.0 0.06 0
- joint femur_tibia_fr: origin xyz=0.0 -0.10 0 -> xyz=0.0 -0.06 0
- joint femur_tibia_rl: origin xyz=0.0 0.10 0 -> xyz=0.0 0.06 0
- joint femur_tibia_rr: origin xyz=0.0 -0.10 0 -> xyz=0.0 -0.06 0

Commit message: Fix demo funs

File: src/envs/bullet_nexabot/quadruped/quadruped.urdf (robot description, URDF)
Before this commit: robot quadruped, 13 links, 12 joints
Joints:
- joint coxa_femur_fl: limit lower=-3 upper=3 effort=100.0 velocity=5 -> lower=-3 upper=3 effort=2.0 velocity=5
- joint coxa_femur_fr: limit lower=-3 upper=3 effort=100.0 velocity=5 -> lower=-3 upper=3 effort=2.0 velocity=5
- joint coxa_femur_rl: limit lower=-3 upper=3 effort=100.0 velocity=5 -> lower=-3 upper=3 effort=2.0 velocity=5
- joint coxa_femur_rr: limit lower=-3 upper=3 effort=100.0 velocity=5 -> lower=-3 upper=3 effort=2.0 velocity=5
- joint femur_tibia_fl: limit lower=-3 upper=3 effort=100.0 velocity=5 -> lower=-3 upper=3 effort=2.0 velocity=5
- joint femur_tibia_fr: limit lower=-3 upper=3 effort=100.0 velocity=5 -> lower=-3 upper=3 effort=2.0 velocity=5
- joint femur_tibia_rl: limit lower=-3 upper=3 effort=100.0 velocity=5 -> lower=-3 upper=3 effort=2.0 velocity=5
- joint femur_tibia_rr: limit lower=-3 upper=3 effort=100.0 velocity=5 -> lower=-3 upper=3 effort=2.0 velocity=5
- joint torso_coxa_fl: limit lower=-3 upper=3 effort=100.0 velocity=5 -> lower=-3 upper=3 effort=2.0 velocity=5
- joint torso_coxa_fr: limit lower=-3 upper=3 effort=100.0 velocity=5 -> lower=-3 upper=3 effort=2.0 velocity=5
- joint torso_coxa_rl: limit lower=-3 upper=3 effort=100.0 velocity=5 -> lower=-3 upper=3 effort=2.0 velocity=5
- joint torso_coxa_rr: limit lower=-3 upper=3 effort=100.0 velocity=5 -> lower=-3 upper=3 effort=2.0 velocity=5

Commit message: Fix demo funs

File: src/envs/bullet_nexabot/quadruped/quadruped.urdf (robot description, URDF)
Before this commit: robot quadruped, 13 links, 12 joints
Joints:
- joint torso_coxa_fl: origin xyz=0.05 0.05 0 -> xyz=0.05 0.05 0 rpy=0 0 -0.7
- joint torso_coxa_fr: origin xyz=0.05 -0.05 0 -> xyz=0.05 -0.05 0 rpy=0 0 0.7
- joint torso_coxa_rl: origin xyz=-0.05 0.05 0 -> xyz=-0.05 0.05 0 rpy=0 0 0.7
- joint torso_coxa_rr: origin xyz=-0.05 -0.05 0 -> xyz=-0.05 -0.05 0 rpy=0 0 -0.7

Commit message: quad env with randomization

File: src/envs/bullet_nexabot/quadruped/quadruped.urdf (robot description, URDF)
Before this commit: robot quadruped, 13 links, 12 joints
Joints:
- joint coxa_femur_fl: origin xyz=0.0 0.01 0 -> xyz=0.0 0.02 0
- joint coxa_femur_fr: origin xyz=0.0 -0.01 0 -> xyz=0.0 -0.02 0
- joint coxa_femur_rl: origin xyz=0.0 0.01 0 -> xyz=0.0 0.02 0
- joint coxa_femur_rr: origin xyz=0.0 -0.01 0 -> xyz=0.0 -0.02 0
