Commit message: PG, ES, SB working

File: src/envs/bullet_quadruped/quadruped.urdf (robot description, URDF)
Before this commit: robot quadruped, 13 links, 12 joints
Joints:
- joint coxa_femur_fl: limit lower=-3 upper=3 effort=2.0 velocity=5 -> lower=-1.8 upper=-0.2 effort=2.0 velocity=5
- joint coxa_femur_fr: limit lower=-3 upper=3 effort=2.0 velocity=5 -> lower=-1.8 upper=-0.2 effort=2.0 velocity=5
- joint coxa_femur_rl: limit lower=-3 upper=3 effort=2.0 velocity=5 -> lower=-1.8 upper=-0.2 effort=2.0 velocity=5
- joint coxa_femur_rr: limit lower=-3 upper=3 effort=2.0 velocity=5 -> lower=-1.8 upper=-0.2 effort=2.0 velocity=5
- joint femur_tibia_fl: limit lower=-3 upper=3 effort=2.0 velocity=5 -> lower=1.4 upper=2.6 effort=2.0 velocity=5
- joint femur_tibia_fr: limit lower=-3 upper=3 effort=2.0 velocity=5 -> lower=1.4 upper=2.6 effort=2.0 velocity=5
- joint femur_tibia_rl: limit lower=-3 upper=3 effort=2.0 velocity=5 -> lower=1.4 upper=2.6 effort=2.0 velocity=5
- joint femur_tibia_rr: limit lower=-3 upper=3 effort=2.0 velocity=5 -> lower=1.4 upper=2.6 effort=2.0 velocity=5
- joint torso_coxa_fl: limit lower=-3 upper=3 effort=2.0 velocity=5 -> lower=-0.5 upper=0.5 effort=2.0 velocity=5
- joint torso_coxa_fr: limit lower=-3 upper=3 effort=2.0 velocity=5 -> lower=-0.5 upper=0.5 effort=2.0 velocity=5
- joint torso_coxa_rl: limit lower=-3 upper=3 effort=2.0 velocity=5 -> lower=-0.5 upper=0.5 effort=2.0 velocity=5
- joint torso_coxa_rr: limit lower=-3 upper=3 effort=2.0 velocity=5 -> lower=-0.5 upper=0.5 effort=2.0 velocity=5
