Commit message: c

File: src/envs/bullet_hexapod/hexapod_legsensor.urdf (robot description, URDF)
Before this commit: robot quadruped, 25 links, 24 joints
Links:
- link coxa_fl: geometry visual cylinder length=0.052 radius=0.015
- link coxa_fr: geometry visual cylinder length=0.052 radius=0.015
- link coxa_ml: geometry visual cylinder length=0.052 radius=0.015
- link coxa_mr: geometry visual cylinder length=0.052 radius=0.015
- link coxa_rl: geometry visual cylinder length=0.052 radius=0.015
- link coxa_rr: geometry visual cylinder length=0.052 radius=0.015
- link tibia_fl: geometry visual cylinder length=0.132 radius=0.015
- link tibia_fr: geometry visual cylinder length=0.132 radius=0.015
- link tibia_ml: geometry visual cylinder length=0.132 radius=0.015
- link tibia_mr: geometry visual cylinder length=0.132 radius=0.015
- link tibia_rl: geometry visual cylinder length=0.132 radius=0.015
- link tibia_rr: geometry visual cylinder length=0.132 radius=0.015
Joints:
- joint tibia_tip_fl: origin xyz=0.0 0.132 0 rpy=0 0 0 -> xyz=0.0 0.112 0 rpy=0 0 0
- joint tibia_tip_fr: origin xyz=0.0 0.132 0 rpy=0 0 0 -> xyz=0.0 0.112 0 rpy=0 0 0
- joint tibia_tip_ml: origin xyz=0.0 0.132 0 rpy=0 0 0 -> xyz=0.0 0.112 0 rpy=0 0 0
- joint tibia_tip_mr: origin xyz=0.0 0.132 0 rpy=0 0 0 -> xyz=0.0 0.112 0 rpy=0 0 0
- joint tibia_tip_rl: origin xyz=0.0 0.132 0 rpy=0 0 0 -> xyz=0.0 0.112 0 rpy=0 0 0
- joint tibia_tip_rr: origin xyz=0.0 0.132 0 rpy=0 0 0 -> xyz=0.0 0.112 0 rpy=0 0 0
