Commit message: c

File: src/envs/bullet_hexapod/hexapod_normal.urdf (robot description, URDF)
Before this commit: robot quadruped, 19 links, 18 joints
Joints:
- joint coxa_femur_fl: limit lower=-1.6 upper=-0.6 effort=1.4 velocity=1 -> lower=-0.5 upper=0.5 effort=1.4 velocity=1
- joint coxa_femur_fr: limit lower=-1.6 upper=-0.6 effort=1.4 velocity=1 -> lower=-0.5 upper=0.5 effort=1.4 velocity=1
- joint coxa_femur_ml: limit lower=-1.6 upper=-0.6 effort=1.4 velocity=1 -> lower=-0.5 upper=0.5 effort=1.4 velocity=1
- joint coxa_femur_mr: limit lower=-1.6 upper=-0.6 effort=1.4 velocity=1 -> lower=-0.5 upper=0.5 effort=1.4 velocity=1
- joint coxa_femur_rl: limit lower=-1.6 upper=-0.6 effort=1.4 velocity=1 -> lower=-0.5 upper=0.5 effort=1.4 velocity=1
- joint coxa_femur_rr: limit lower=-1.6 upper=-0.6 effort=1.4 velocity=1 -> lower=-0.5 upper=0.5 effort=1.4 velocity=1
- joint femur_tibia_fl: limit lower=0.9 upper=1.9 effort=1.4 velocity=1 -> lower=0.7 upper=1.7 effort=1.4 velocity=1
- joint femur_tibia_fr: limit lower=0.9 upper=1.9 effort=1.4 velocity=1 -> lower=0.7 upper=1.7 effort=1.4 velocity=1
- joint femur_tibia_ml: limit lower=0.9 upper=1.9 effort=1.4 velocity=1 -> lower=0.7 upper=1.7 effort=1.4 velocity=1
- joint femur_tibia_mr: limit lower=0.9 upper=1.9 effort=1.4 velocity=1 -> lower=0.7 upper=1.7 effort=1.4 velocity=1
- joint femur_tibia_rl: limit lower=0.9 upper=1.9 effort=1.4 velocity=1 -> lower=0.7 upper=1.7 effort=1.4 velocity=1
- joint femur_tibia_rr: limit lower=0.9 upper=1.9 effort=1.4 velocity=1 -> lower=0.7 upper=1.7 effort=1.4 velocity=1

File: src/envs/bullet_hexapod/hexapod_wide_range.urdf (robot description, URDF)
Before this commit: robot quadruped, 19 links, 18 joints
Joints:
- joint coxa_femur_fl: limit lower=-5.0 upper=5.0 effort=1.4 velocity=1 -> lower=-0.5 upper=0.5 effort=1.4 velocity=1
- joint coxa_femur_fr: limit lower=-5.0 upper=5.0 effort=1.4 velocity=1 -> lower=-0.5 upper=0.5 effort=1.4 velocity=1
- joint coxa_femur_ml: limit lower=-5.0 upper=5.0 effort=1.4 velocity=1 -> lower=-0.5 upper=0.5 effort=1.4 velocity=1
- joint coxa_femur_mr: limit lower=-5.0 upper=5.0 effort=1.4 velocity=1 -> lower=-0.5 upper=0.5 effort=1.4 velocity=1
- joint coxa_femur_rl: limit lower=-5.0 upper=5.0 effort=1.4 velocity=1 -> lower=-0.5 upper=0.5 effort=1.4 velocity=1
- joint coxa_femur_rr: limit lower=-5.0 upper=5.0 effort=1.4 velocity=1 -> lower=-0.5 upper=0.5 effort=1.4 velocity=1
- joint femur_tibia_fl: limit lower=-5.0 upper=5.0 effort=1.4 velocity=1 -> lower=0.7 upper=1.7 effort=1.4 velocity=1
- joint femur_tibia_fr: limit lower=-5.0 upper=5.0 effort=1.4 velocity=1 -> lower=0.7 upper=1.7 effort=1.4 velocity=1
- joint femur_tibia_ml: limit lower=-5.0 upper=5.0 effort=1.4 velocity=1 -> lower=0.7 upper=1.7 effort=1.4 velocity=1
- joint femur_tibia_mr: limit lower=-5.0 upper=5.0 effort=1.4 velocity=1 -> lower=0.7 upper=1.7 effort=1.4 velocity=1
- joint femur_tibia_rl: limit lower=-5.0 upper=5.0 effort=1.4 velocity=1 -> lower=0.7 upper=1.7 effort=1.4 velocity=1
- joint femur_tibia_rr: limit lower=-5.0 upper=5.0 effort=1.4 velocity=1 -> lower=0.7 upper=1.7 effort=1.4 velocity=1
- joint torso_coxa_fl: limit lower=-5.0 upper=5.0 effort=1.4 velocity=1 -> lower=-0.4 upper=0.4 effort=1.4 velocity=1
- joint torso_coxa_fr: limit lower=-5.0 upper=5.0 effort=1.4 velocity=1 -> lower=-0.4 upper=0.4 effort=1.4 velocity=1
- joint torso_coxa_ml: limit lower=-5.0 upper=5.0 effort=1.4 velocity=1 -> lower=-0.4 upper=0.4 effort=1.4 velocity=1
- joint torso_coxa_mr: limit lower=-5.0 upper=5.0 effort=1.4 velocity=1 -> lower=-0.4 upper=0.4 effort=1.4 velocity=1
- joint torso_coxa_rl: limit lower=-5.0 upper=5.0 effort=1.4 velocity=1 -> lower=-0.4 upper=0.4 effort=1.4 velocity=1
- joint torso_coxa_rr: limit lower=-5.0 upper=5.0 effort=1.4 velocity=1 -> lower=-0.4 upper=0.4 effort=1.4 velocity=1

Commit message: c

File: src/envs/bullet_hexapod/hexapod_normal.urdf (robot description, URDF)
Before this commit: robot quadruped, 19 links, 18 joints
Joints:
- joint coxa_femur_fl: limit lower=-0.5 upper=0.5 effort=1.4 velocity=1 -> lower=-0.7 upper=0.7 effort=1.4 velocity=1
- joint coxa_femur_fr: limit lower=-0.5 upper=0.5 effort=1.4 velocity=1 -> lower=-0.7 upper=0.7 effort=1.4 velocity=1
- joint coxa_femur_ml: limit lower=-0.5 upper=0.5 effort=1.4 velocity=1 -> lower=-0.7 upper=0.7 effort=1.4 velocity=1
- joint coxa_femur_mr: limit lower=-0.5 upper=0.5 effort=1.4 velocity=1 -> lower=-0.7 upper=0.7 effort=1.4 velocity=1
- joint coxa_femur_rl: limit lower=-0.5 upper=0.5 effort=1.4 velocity=1 -> lower=-0.7 upper=0.7 effort=1.4 velocity=1
- joint coxa_femur_rr: limit lower=-0.5 upper=0.5 effort=1.4 velocity=1 -> lower=-0.7 upper=0.7 effort=1.4 velocity=1
- joint femur_tibia_fl: limit lower=0.7 upper=1.7 effort=1.4 velocity=1 -> lower=0.5 upper=1.4 effort=1.4 velocity=1
- joint femur_tibia_fr: limit lower=0.7 upper=1.7 effort=1.4 velocity=1 -> lower=0.5 upper=1.4 effort=1.4 velocity=1
- joint femur_tibia_ml: limit lower=0.7 upper=1.7 effort=1.4 velocity=1 -> lower=0.5 upper=1.4 effort=1.4 velocity=1
- joint femur_tibia_mr: limit lower=0.7 upper=1.7 effort=1.4 velocity=1 -> lower=0.5 upper=1.4 effort=1.4 velocity=1
- joint femur_tibia_rl: limit lower=0.7 upper=1.7 effort=1.4 velocity=1 -> lower=0.5 upper=1.4 effort=1.4 velocity=1
- joint femur_tibia_rr: limit lower=0.7 upper=1.7 effort=1.4 velocity=1 -> lower=0.5 upper=1.4 effort=1.4 velocity=1

Commit message: c

File: src/envs/bullet_hexapod/hexapod_normal.urdf (robot description, URDF)
Before this commit: robot quadruped, 19 links, 18 joints
Joints:
- joint coxa_femur_fl: limit lower=-0.7 upper=0.7 effort=1.4 velocity=1 -> lower=-0.9 upper=0.7 effort=1.4 velocity=1
- joint coxa_femur_fr: limit lower=-0.7 upper=0.7 effort=1.4 velocity=1 -> lower=-0.9 upper=0.7 effort=1.4 velocity=1
- joint coxa_femur_ml: limit lower=-0.7 upper=0.7 effort=1.4 velocity=1 -> lower=-0.9 upper=0.7 effort=1.4 velocity=1
- joint coxa_femur_mr: limit lower=-0.7 upper=0.7 effort=1.4 velocity=1 -> lower=-0.9 upper=0.7 effort=1.4 velocity=1
- joint coxa_femur_rl: limit lower=-0.7 upper=0.7 effort=1.4 velocity=1 -> lower=-0.9 upper=0.7 effort=1.4 velocity=1
- joint coxa_femur_rr: limit lower=-0.7 upper=0.7 effort=1.4 velocity=1 -> lower=-0.9 upper=0.7 effort=1.4 velocity=1
- joint femur_tibia_fl: limit lower=0.5 upper=1.4 effort=1.4 velocity=1 -> lower=0.2 upper=1.4 effort=1.4 velocity=1
- joint femur_tibia_fr: limit lower=0.5 upper=1.4 effort=1.4 velocity=1 -> lower=0.2 upper=1.4 effort=1.4 velocity=1
- joint femur_tibia_ml: limit lower=0.5 upper=1.4 effort=1.4 velocity=1 -> lower=0.2 upper=1.4 effort=1.4 velocity=1
- joint femur_tibia_mr: limit lower=0.5 upper=1.4 effort=1.4 velocity=1 -> lower=0.2 upper=1.4 effort=1.4 velocity=1
- joint femur_tibia_rl: limit lower=0.5 upper=1.4 effort=1.4 velocity=1 -> lower=0.2 upper=1.4 effort=1.4 velocity=1
- joint femur_tibia_rr: limit lower=0.5 upper=1.4 effort=1.4 velocity=1 -> lower=0.2 upper=1.4 effort=1.4 velocity=1
- joint torso_coxa_fl: limit lower=-0.4 upper=0.4 effort=1.4 velocity=1 -> lower=-0.5 upper=0.5 effort=1.4 velocity=1
- joint torso_coxa_fr: limit lower=-0.4 upper=0.4 effort=1.4 velocity=1 -> lower=-0.5 upper=0.5 effort=1.4 velocity=1
- joint torso_coxa_ml: limit lower=-0.4 upper=0.4 effort=1.4 velocity=1 -> lower=-0.5 upper=0.5 effort=1.4 velocity=1
- joint torso_coxa_mr: limit lower=-0.4 upper=0.4 effort=1.4 velocity=1 -> lower=-0.5 upper=0.5 effort=1.4 velocity=1
- joint torso_coxa_rl: limit lower=-0.4 upper=0.4 effort=1.4 velocity=1 -> lower=-0.5 upper=0.5 effort=1.4 velocity=1
- joint torso_coxa_rr: limit lower=-0.4 upper=0.4 effort=1.4 velocity=1 -> lower=-0.5 upper=0.5 effort=1.4 velocity=1

Commit message: c

File: src/envs/bullet_hexapod/hexapod_normal.urdf (robot description, URDF)
Before this commit: robot quadruped, 19 links, 18 joints
Joints:
- joint coxa_femur_fl: limit lower=-0.9 upper=0.7 effort=1.4 velocity=1 -> lower=-3.0 upper=3.0 effort=1.4 velocity=1
- joint coxa_femur_fr: limit lower=-0.9 upper=0.7 effort=1.4 velocity=1 -> lower=-3.0 upper=3.0 effort=1.4 velocity=1
- joint coxa_femur_ml: limit lower=-0.9 upper=0.7 effort=1.4 velocity=1 -> lower=-3.0 upper=3.0 effort=1.4 velocity=1
- joint coxa_femur_mr: limit lower=-0.9 upper=0.7 effort=1.4 velocity=1 -> lower=-3.0 upper=3.0 effort=1.4 velocity=1
- joint coxa_femur_rl: limit lower=-0.9 upper=0.7 effort=1.4 velocity=1 -> lower=-3.0 upper=3.0 effort=1.4 velocity=1
- joint coxa_femur_rr: limit lower=-0.9 upper=0.7 effort=1.4 velocity=1 -> lower=-3.0 upper=3.0 effort=1.4 velocity=1
- joint femur_tibia_fl: limit lower=0.2 upper=1.4 effort=1.4 velocity=1 -> lower=-3.0 upper=3.0 effort=1.4 velocity=1
- joint femur_tibia_fr: limit lower=0.2 upper=1.4 effort=1.4 velocity=1 -> lower=-3.0 upper=3.0 effort=1.4 velocity=1
- joint femur_tibia_ml: limit lower=0.2 upper=1.4 effort=1.4 velocity=1 -> lower=-3.0 upper=3.0 effort=1.4 velocity=1
- joint femur_tibia_mr: limit lower=0.2 upper=1.4 effort=1.4 velocity=1 -> lower=-3.0 upper=3.0 effort=1.4 velocity=1
- joint femur_tibia_rl: limit lower=0.2 upper=1.4 effort=1.4 velocity=1 -> lower=-3.0 upper=3.0 effort=1.4 velocity=1
- joint femur_tibia_rr: limit lower=0.2 upper=1.4 effort=1.4 velocity=1 -> lower=-3.0 upper=3.0 effort=1.4 velocity=1
- joint torso_coxa_fl: limit lower=-0.5 upper=0.5 effort=1.4 velocity=1 -> lower=-3.0 upper=3.0 effort=1.4 velocity=1
- joint torso_coxa_fr: limit lower=-0.5 upper=0.5 effort=1.4 velocity=1 -> lower=-3.0 upper=3.0 effort=1.4 velocity=1
- joint torso_coxa_ml: limit lower=-0.5 upper=0.5 effort=1.4 velocity=1 -> lower=-3.0 upper=3.0 effort=1.4 velocity=1
- joint torso_coxa_mr: limit lower=-0.5 upper=0.5 effort=1.4 velocity=1 -> lower=-3.0 upper=3.0 effort=1.4 velocity=1
- joint torso_coxa_rl: limit lower=-0.5 upper=0.5 effort=1.4 velocity=1 -> lower=-3.0 upper=3.0 effort=1.4 velocity=1
- joint torso_coxa_rr: limit lower=-0.5 upper=0.5 effort=1.4 velocity=1 -> lower=-3.0 upper=3.0 effort=1.4 velocity=1

Commit message: c

File: src/envs/bullet_hexapod/hexapod_normal.urdf (robot description, URDF)
Before this commit: robot quadruped, 19 links, 18 joints
Joints:
- joint coxa_femur_fl: limit lower=-3.0 upper=3.0 effort=1.4 velocity=1 -> lower=-6.0 upper=6.0 effort=1.4 velocity=1
- joint coxa_femur_fr: limit lower=-3.0 upper=3.0 effort=1.4 velocity=1 -> lower=-6.0 upper=6.0 effort=1.4 velocity=1
- joint coxa_femur_ml: limit lower=-3.0 upper=3.0 effort=1.4 velocity=1 -> lower=-6.0 upper=6.0 effort=1.4 velocity=1
- joint coxa_femur_mr: limit lower=-3.0 upper=3.0 effort=1.4 velocity=1 -> lower=-6.0 upper=6.0 effort=1.4 velocity=1
- joint coxa_femur_rl: limit lower=-3.0 upper=3.0 effort=1.4 velocity=1 -> lower=-6.0 upper=6.0 effort=1.4 velocity=1
- joint coxa_femur_rr: limit lower=-3.0 upper=3.0 effort=1.4 velocity=1 -> lower=-6.0 upper=6.0 effort=1.4 velocity=1
- joint femur_tibia_fl: limit lower=-3.0 upper=3.0 effort=1.4 velocity=1 -> lower=-6.0 upper=6.0 effort=1.4 velocity=1
- joint femur_tibia_fr: limit lower=-3.0 upper=3.0 effort=1.4 velocity=1 -> lower=-6.0 upper=6.0 effort=1.4 velocity=1
- joint femur_tibia_ml: limit lower=-3.0 upper=3.0 effort=1.4 velocity=1 -> lower=-6.0 upper=6.0 effort=1.4 velocity=1
- joint femur_tibia_mr: limit lower=-3.0 upper=3.0 effort=1.4 velocity=1 -> lower=-6.0 upper=6.0 effort=1.4 velocity=1
- joint femur_tibia_rl: limit lower=-3.0 upper=3.0 effort=1.4 velocity=1 -> lower=-6.0 upper=6.0 effort=1.4 velocity=1
- joint femur_tibia_rr: limit lower=-3.0 upper=3.0 effort=1.4 velocity=1 -> lower=-6.0 upper=6.0 effort=1.4 velocity=1
- joint torso_coxa_fl: limit lower=-3.0 upper=3.0 effort=1.4 velocity=1 -> lower=-6.0 upper=6.0 effort=1.4 velocity=1
- joint torso_coxa_fr: limit lower=-3.0 upper=3.0 effort=1.4 velocity=1 -> lower=-6.0 upper=6.0 effort=1.4 velocity=1
- joint torso_coxa_ml: limit lower=-3.0 upper=3.0 effort=1.4 velocity=1 -> lower=-6.0 upper=6.0 effort=1.4 velocity=1
- joint torso_coxa_mr: limit lower=-3.0 upper=3.0 effort=1.4 velocity=1 -> lower=-6.0 upper=6.0 effort=1.4 velocity=1
- joint torso_coxa_rl: limit lower=-3.0 upper=3.0 effort=1.4 velocity=1 -> lower=-6.0 upper=6.0 effort=1.4 velocity=1
- joint torso_coxa_rr: limit lower=-3.0 upper=3.0 effort=1.4 velocity=1 -> lower=-6.0 upper=6.0 effort=1.4 velocity=1

Commit message: c

File: src/envs/bullet_hexapod/hexapod_normal.urdf (robot description, URDF)
Before this commit: robot quadruped, 19 links, 18 joints
Links:
- link torso: geometry collision box size=0.20 0.12 0.01; visual box size=0.20 0.12 0.01

Commit message: Working on perlin oscillator policy

File: src/envs/bullet_hexapod/hexapod_normal.urdf (robot description, URDF)
Before this commit: robot quadruped, 19 links, 18 joints
Links:
- link torso: geometry collision box size=0.20 0.12 0.03; visual box size=0.20 0.12 0.03

Commit message: c

File: src/envs/bullet_hexapod/hexapod_normal.urdf (robot description, URDF)
Before this commit: robot quadruped, 19 links, 18 joints
Links:
- link torso: geometry collision box size=0.20 0.12 0.06; visual box size=0.20 0.12 0.06
