Commit message: c

File: src/envs/bullet_quadrotor/quadrotor_rnd.urdf (robot description, URDF)
Before this commit: robot quadrotor, 9 links, 8 joints
Links:
- link boom_fl: geometry visual cylinder length=0.39593001059648625 radius=0.015
- link boom_fr: geometry visual cylinder length=0.39593001059648625 radius=0.015
- link boom_rl: geometry visual cylinder length=0.39593001059648625 radius=0.015
- link boom_rr: geometry visual cylinder length=0.39593001059648625 radius=0.015
Joints:
- joint boom_motor_fl: origin xyz=0 0.5067586307404879 0 rpy=0 0 0 -> xyz=0 0.39593001059648625 0 rpy=0 0 0
- joint boom_motor_fr: origin xyz=0 0.5067586307404879 0 rpy=0 0 0 -> xyz=0 0.39593001059648625 0 rpy=0 0 0
- joint boom_motor_rl: origin xyz=0 0.5067586307404879 0 rpy=0 0 0 -> xyz=0 0.39593001059648625 0 rpy=0 0 0
- joint boom_motor_rr: origin xyz=0 0.5067586307404879 0 rpy=0 0 0 -> xyz=0 0.39593001059648625 0 rpy=0 0 0

Commit message: c

File: src/envs/bullet_quadrotor/quadrotor_rnd.urdf (robot description, URDF)
Before this commit: robot quadrotor, 9 links, 8 joints
Links:
- link boom_fl: geometry visual cylinder length=0.17258571375788076 radius=0.015
- link boom_fr: geometry visual cylinder length=0.17258571375788076 radius=0.015
- link boom_rl: geometry visual cylinder length=0.17258571375788076 radius=0.015
- link boom_rr: geometry visual cylinder length=0.17258571375788076 radius=0.015
Joints:
- joint boom_motor_fl: origin xyz=0 0.39593001059648625 0 rpy=0 0 0 -> xyz=0 0.17258571375788076 0 rpy=0 0 0
- joint boom_motor_fr: origin xyz=0 0.39593001059648625 0 rpy=0 0 0 -> xyz=0 0.17258571375788076 0 rpy=0 0 0
- joint boom_motor_rl: origin xyz=0 0.39593001059648625 0 rpy=0 0 0 -> xyz=0 0.17258571375788076 0 rpy=0 0 0
- joint boom_motor_rr: origin xyz=0 0.39593001059648625 0 rpy=0 0 0 -> xyz=0 0.17258571375788076 0 rpy=0 0 0

Commit message: c

File: src/envs/bullet_quadrotor/quadrotor_rnd.urdf (robot description, URDF)
Before this commit: robot quadrotor, 9 links, 8 joints
Links:
- link boom_fl: geometry visual cylinder length=0.49171169135321313 radius=0.015
- link boom_fr: geometry visual cylinder length=0.49171169135321313 radius=0.015
- link boom_rl: geometry visual cylinder length=0.49171169135321313 radius=0.015
- link boom_rr: geometry visual cylinder length=0.49171169135321313 radius=0.015
Joints:
- joint boom_motor_fl: origin xyz=0 0.17258571375788076 0 rpy=0 0 0 -> xyz=0 0.49171169135321313 0 rpy=0 0 0
- joint boom_motor_fr: origin xyz=0 0.17258571375788076 0 rpy=0 0 0 -> xyz=0 0.49171169135321313 0 rpy=0 0 0
- joint boom_motor_rl: origin xyz=0 0.17258571375788076 0 rpy=0 0 0 -> xyz=0 0.49171169135321313 0 rpy=0 0 0
- joint boom_motor_rr: origin xyz=0 0.17258571375788076 0 rpy=0 0 0 -> xyz=0 0.49171169135321313 0 rpy=0 0 0

Commit message: c

File: src/envs/bullet_quadrotor/quadrotor_rnd.urdf (robot description, URDF)
Before this commit: robot quadrotor, 9 links, 8 joints
Links:
- link boom_fl: geometry visual cylinder length=0.2 radius=0.015
- link boom_fr: geometry visual cylinder length=0.2 radius=0.015
- link boom_rl: geometry visual cylinder length=0.2 radius=0.015
- link boom_rr: geometry visual cylinder length=0.2 radius=0.015
Joints:
- joint boom_motor_fl: origin xyz=0 0.49171169135321313 0 rpy=0 0 0 -> xyz=0 0.2 0 rpy=0 0 0
- joint boom_motor_fr: origin xyz=0 0.49171169135321313 0 rpy=0 0 0 -> xyz=0 0.2 0 rpy=0 0 0
- joint boom_motor_rl: origin xyz=0 0.49171169135321313 0 rpy=0 0 0 -> xyz=0 0.2 0 rpy=0 0 0
- joint boom_motor_rr: origin xyz=0 0.49171169135321313 0 rpy=0 0 0 -> xyz=0 0.2 0 rpy=0 0 0

Commit message: c

File: src/envs/bullet_quadrotor/quadrotor_rnd.urdf (robot description, URDF)
Before this commit: robot quadrotor, 9 links, 8 joints
Links:
- link boom_fl: geometry visual cylinder length=0.3914990906203317 radius=0.015
- link boom_fr: geometry visual cylinder length=0.3914990906203317 radius=0.015
- link boom_rl: geometry visual cylinder length=0.3914990906203317 radius=0.015
- link boom_rr: geometry visual cylinder length=0.3914990906203317 radius=0.015
Joints:
- joint boom_motor_fl: origin xyz=0 0.2 0 rpy=0 0 0 -> xyz=0 0.3914990906203317 0 rpy=0 0 0
- joint boom_motor_fr: origin xyz=0 0.2 0 rpy=0 0 0 -> xyz=0 0.3914990906203317 0 rpy=0 0 0
- joint boom_motor_rl: origin xyz=0 0.2 0 rpy=0 0 0 -> xyz=0 0.3914990906203317 0 rpy=0 0 0
- joint boom_motor_rr: origin xyz=0 0.2 0 rpy=0 0 0 -> xyz=0 0.3914990906203317 0 rpy=0 0 0
