Commit message: Made eval for model learning, need to test

File: src/envs/bullet_quadrotor/quadrotor.urdf (robot description, URDF)
Before this commit: robot quadrotor, 9 links, 8 joints
Joints:
- joint base_boom_fr: origin xyz=0.0 0.0 0 rpy=0 0 -0.7854 -> xyz=0.0 0.0 0 rpy=0 0 -2.3562
- joint base_boom_rr: limit lower=-3 upper=3 effort=1.4 velocity=1 -> (none); origin xyz=0.0 0.0 0 rpy=0 0 2.3562 -> xyz=0.0 0.0 0 rpy=0 0 0
- joint boom_motor_fl: child boom_fl -> motor_fl; parent base -> boom_fl
- joint boom_motor_fr: child boom_fr -> motor_fr; parent base -> boom_fr
- joint boom_motor_rl: child boom_rl -> motor_rl; origin xyz=0.0 0.2 0 rpy=0 0 -0.7854 -> xyz=0.0 0.2 0 rpy=0 0 0; parent base -> boom_rl
- joint boom_motor_rr: child boom_rr -> motor_rr; parent base -> boom_rr

Commit message: Made eval for model learning, need to test

File: src/envs/bullet_quadrotor/quadrotor.urdf (robot description, URDF)
Before this commit: robot quadrotor, 9 links, 8 joints
Joints:
- joint base_boom_rr: origin xyz=0.0 0.0 0 rpy=0 0 0 -> xyz=0.0 0.0 0 rpy=0 0 2.3562
- joint boom_motor_rr: origin xyz=0.0 0.2 0 rpy=0 0 -0.7854 -> xyz=0.0 0.2 0 rpy=0 0 0

Commit message: c

File: src/envs/bullet_quadrotor/quadrotor.urdf (robot description, URDF)
Before this commit: robot quadrotor, 9 links, 8 joints
Links:
- link boom_fl: geometry visual cylinder length=0.15 radius=0.015
- link boom_fr: geometry visual cylinder length=0.15 radius=0.015
- link boom_rl: geometry visual cylinder length=0.15 radius=0.015
- link boom_rr: geometry visual cylinder length=0.15 radius=0.015
Joints:
- joint boom_motor_fl: origin xyz=0.0 0.2 0 rpy=0 0 0 -> xyz=0 0.15 0 rpy=0 0 0
- joint boom_motor_fr: origin xyz=0.0 0.2 0 rpy=0 0 0 -> xyz=0 0.15 0 rpy=0 0 0
- joint boom_motor_rl: origin xyz=0.0 0.2 0 rpy=0 0 0 -> xyz=0 0.15 0 rpy=0 0 0
- joint boom_motor_rr: origin xyz=0.0 0.2 0 rpy=0 0 0 -> xyz=0 0.15 0 rpy=0 0 0

File: src/envs/bullet_quadrotor/quadrotor_rnd.urdf (robot description, URDF)
Before this commit: robot quadrotor, 9 links, 8 joints
Links:
- link boom_fl: geometry visual cylinder length=0.15 radius=0.015
- link boom_fr: geometry visual cylinder length=0.15 radius=0.015
- link boom_rl: geometry visual cylinder length=0.15 radius=0.015
- link boom_rr: geometry visual cylinder length=0.15 radius=0.015
Joints:
- joint boom_motor_fl: origin xyz=0 0.3914990906203317 0 rpy=0 0 0 -> xyz=0 0.15 0 rpy=0 0 0
- joint boom_motor_fr: origin xyz=0 0.3914990906203317 0 rpy=0 0 0 -> xyz=0 0.15 0 rpy=0 0 0
- joint boom_motor_rl: origin xyz=0 0.3914990906203317 0 rpy=0 0 0 -> xyz=0 0.15 0 rpy=0 0 0
- joint boom_motor_rr: origin xyz=0 0.3914990906203317 0 rpy=0 0 0 -> xyz=0 0.15 0 rpy=0 0 0
