Commit message: c

File: src/envs/bullet_quadrotor/quadrotor_default_generated.urdf (robot description, URDF)
Before this commit: robot quadrotor, 9 links, 8 joints
Links:
- link boom_fl: geometry visual cylinder length=0.2 radius=0.015
- link boom_fr: geometry visual cylinder length=0.2 radius=0.015
- link boom_rl: geometry visual cylinder length=0.2 radius=0.015
- link boom_rr: geometry visual cylinder length=0.2 radius=0.015
Joints:
- joint boom_motor_fl: origin xyz=0 0.15 0 rpy=0 0 0 -> xyz=0 0.2 0 rpy=0 0 0
- joint boom_motor_fr: origin xyz=0 0.15 0 rpy=0 0 0 -> xyz=0 0.2 0 rpy=0 0 0
- joint boom_motor_rl: origin xyz=0 0.15 0 rpy=0 0 0 -> xyz=0 0.2 0 rpy=0 0 0
- joint boom_motor_rr: origin xyz=0 0.15 0 rpy=0 0 0 -> xyz=0 0.2 0 rpy=0 0 0
